Commit message: feat(project):new version upload

File: diploma_ws/src/runner_sim/models/runner.urdf.xacro (robot description, xacro)
@@ -17,4 +17,9 @@
   <xacro:property name="imu_accel_noise" value="0.02"/>
   <xacro:property name="imu_gyro_noise" value="0.01"/>
+  <!-- Chassis collision starts above the floor so only wheels and casters touch the ground. -->
+  <xacro:property name="ground_clearance" value="0.06"/>
+  <xacro:property name="caster_radius" value="0.09"/>
+  <!-- Casters hang slightly above the floor so the drive wheels always carry the load (traction). -->
+  <xacro:property name="caster_gap" value="0.005"/>
   <material name="runner_blue"><color rgba="0.12 0.32 0.62 1.0"/></material>
   <material name="rubber"><color rgba="0.03 0.03 0.03 1.0"/></material>
@@ -32,6 +37,6 @@
     </visual>
     <collision name="chassis_collision">
-      <origin xyz="0 0 ${body_z}"/>
-      <geometry><box size="${body_length} ${body_width} ${body_height}"/></geometry>
+      <origin xyz="0 0 ${(body_height + ground_clearance) / 2}"/>
+      <geometry><box size="${body_length} ${body_width} ${body_height - ground_clearance}"/></geometry>
     </collision>
   </link>
@@ -56,13 +61,21 @@
     <axis xyz="0 1 0"/>
   </joint>
-  <link name="caster_link">
-    <inertial><mass value="0.8"/><inertia ixx="0.005" iyy="0.005" izz="0.005" ixy="0" ixz="0" iyz="0"/></inertial>
-    <visual><geometry><sphere radius="0.09"/></geometry><material name="rubber"/></visual>
-    <collision><geometry><sphere radius="0.09"/></geometry></collision>
-  </link>
-  <joint name="caster_joint" type="fixed">
-    <parent link="base_link"/><child link="caster_link"/>
-    <origin xyz="0.38 0 0.09"/>
-  </joint>
+  <gazebo reference="left_wheel_link"><mu1>1.0</mu1><mu2>1.0</mu2></gazebo>
+  <gazebo reference="right_wheel_link"><mu1>1.0</mu1><mu2>1.0</mu2></gazebo>
+  <!-- Passive casters are modelled as frictionless spheres, otherwise they brake turning in place. -->
+  <xacro:macro name="caster" params="name x">
+    <link name="${name}_link">
+      <inertial><mass value="0.8"/><inertia ixx="0.005" iyy="0.005" izz="0.005" ixy="0" ixz="0" iyz="0"/></inertial>
+      <visual><geometry><sphere radius="${caster_radius}"/></geometry><material name="rubber"/></visual>
+      <collision><geometry><sphere radius="${caster_radius}"/></geometry></collision>
+    </link>
+    <joint name="${name}_joint" type="fixed">
+      <parent link="base_link"/><child link="${name}_link"/>
+      <origin xyz="${x} 0 ${caster_radius + caster_gap}"/>
+    </joint>
+    <gazebo reference="${name}_link"><mu1>0.0</mu1><mu2>0.0</mu2></gazebo>
+  </xacro:macro>
+  <xacro:caster name="front_caster" x="0.38"/>
+  <xacro:caster name="rear_caster" x="-0.38"/>
   <xacro:macro name="lidar" params="name x y yaw topic">
     <link name="${name}_link">
@@ -109,4 +122,9 @@
       <max_linear_velocity>2.0</max_linear_velocity>
       <max_angular_velocity>1.5707963267948966</max_angular_velocity>
+      <!-- Without acceleration limits velocity steps make the wheels slip and corrupt wheel odometry. -->
+      <min_linear_acceleration>-1.0</min_linear_acceleration>
+      <max_linear_acceleration>1.0</max_linear_acceleration>
+      <min_angular_acceleration>-2.0</min_angular_acceleration>
+      <max_angular_acceleration>2.0</max_angular_acceleration>
       <topic>/$(arg robot_name)/cmd_vel</topic>
       <odom_topic>/$(arg robot_name)/wheel/odometry</odom_topic>
